File: applications/2dimmer_4te/Dimmer_1.3.brd (EAGLE design)
At the start: 87.3 x 67.3 mm, 41 parts, among them IC1 CNY17, IC2 89LPC922, IC3 CNY17, IC4 CNY17, K1 ISP, Q1 IRFP460, Q2 IRFP460, Q3 IRFP460, Q4 IRFP460

Commit message: 2,2nF mit X2 gekennzeichnet
Parts:
- C2: value 2,2nF -> 2,2nF X2
Changed lines of the file:
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@@
 <element name="R8" library="rcl" package="0204/7" value="100k" x="36.195" y="34.29" rot="R180"/>
 <element name="R9" library="rcl" package="0204/7" value="100k" x="36.195" y="45.72" rot="R180"/>
-<element name="C2" library="rcl" package="C075-063X106" value="2,2nF" x="46.99" y="31.115" rot="R180"/>
+<element name="C2" library="rcl" package="C075-063X106" value="2,2nF X2" x="46.99" y="31.115" rot="R180"/>
 <element name="D3" library="diode" package="DO35-10" value="1N4007" x="50.8" y="36.195"/>
 <element name="R15" library="rcl" package="0204/7" value="100k" x="41.91" y="38.1" rot="R180"/>
