File: applications/Torsteuerung/Torsteuerung_1.0.sch (EAGLE design)
At the start: 77 parts, among them IC1 74HC14N, IC2 74HC14N

Commit message: Tasterschnittstelle_DIL übersiedelte nach UPModule
Parts:
- R14, R15: device rcl:R-EU_0207/2V -> rcl:R-EU_0204/5
Changed lines of the file:
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@@
 <part name="OK7" library="optocoupler" deviceset="CNY17" device=""/>
 <part name="OK8" library="optocoupler" deviceset="CNY17" device=""/>
-<part name="R14" library="rcl" deviceset="R-EU_" device="0207/2V" value="330"/>
-<part name="R15" library="rcl" deviceset="R-EU_" device="0207/2V" value="330"/>
+<part name="R14" library="rcl" deviceset="R-EU_" device="0204/5" value="330"/>
+<part name="R15" library="rcl" deviceset="R-EU_" device="0204/5" value="330"/>
 <part name="GND10" library="supply1" deviceset="GND" device=""/>
 <part name="GND11" library="supply1" deviceset="GND" device=""/>
