File: modules/UPModule/SB_TS_1.54.brd (EAGLE design)
At the start: 42.3 x 27.4 mm, 67 parts, among them IC1 MC34063AD, IC2 MCP1702-33, Q1 BC856, Q2 BCP52, T1 BC848, T2 BC848, U1 89LPC922

Commit message: version 2.53 gelöscht und kerkobug 10nF am OSC von 1.54 gefixt.
Parts:
- C8: value 10pf -> 10nf
Changed lines of the file:
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@@
 <attribute name="VALUE" x="8.0963" y="17.7008" size="1.27" layer="28" rot="MR180"/>
 </element>
-<element name="C8" library="rcl" package="C1206" value="10pf" x="20.5113" y="16.17795" smashed="yes" rot="MR270">
+<element name="C8" library="rcl" package="C1206" value="10nf" x="20.5113" y="16.17795" smashed="yes" rot="MR270">
 <attribute name="NAME" x="20.3526" y="17.36865" size="1.27" layer="26" rot="MR270"/>
 <attribute name="VALUE" x="22.3369" y="18.16235" size="1.27" layer="28" rot="MR270"/>
