File: modules/UPModule/TS-ARM3.0_8.brd (EAGLE design)
At the start: 42.3 x 27.4 mm, 80 parts, among them IC1 LPC1115, IC100 BD9G101, P1 , P10 , P11 , P12 , P13 , P14 , P2 , P3 , P4 , P5 , P6 , P7 , P8 , P9 , T1 BC856, T2 BCP52, T3 BC847, X1 EIB

Commit message: overlap beseitigt
Routing:
- net GND: track 83.1 -> 85.0 mm
- net BUS_V: track 47.9 -> 47.3 mm
