File: modules/UPModule/UP-Module-fused-IOs.sch (EAGLE design)
At the start: 137 parts, among them IC1 LPC1115, IC100 BD9G101, IC2 ESDA5V3L, IC302 ESDA5V3L, IC303 ESDA5V3L, IC304 ESDA5V3L, IC401 ESDA5V3L, IC402 ESDA5V3L, IC403 ESDA5V3L, IC404 ESDA5V3L, Q2 ASFL, T1 BC856, T2 BCP52, T3 BC847, X1 EIB, X2 B7B-PH-K-S, X3 B8B-PH-K-S

Commit message: Update of UP Module with fused IOs
Completely changed how IOs will be protected. EEPROM and cropty IC added.
Parts:
- removed C302.1, C302.2, C303.1, C303.2, C304.1, C304.2, C304.3, C304.4, C401.1, C401.2, C402.1, C402.2, C403.1, C403.2, C404.1, C404.2: 10nF/50V, rcl:C-EUC0805
- removed F13, F14, F15, F16, F3, F4, F5: BSMD0805-005-33V, rcl:R-EU_R0805
- removed IC2, IC302, IC303, IC304, IC401, IC402, IC403, IC404: ESDA5V3L, SamacSys_Parts:ESDA5V3L
- removed R302.1, R302.2, R303.1, R303.2, R304.1, R304.2, R304.5, R304.6, R401.1, R401.2, R402.1, R402.2, R403.1, R403.2, R404.1, R404.2: 1M, rcl:R-EU_R0805
- removed R302.3, R302.4, R303.3, R303.4, R304.3, R304.4, R304.7, R304.8, R401.3, R401.4, R402.3, R402.4, R403.3, R403.4, R404.3, R404.4: 1k, rcl:R-EU_R0805
- removed STECKER1, STECKER2: B12B-PH-K-S, con-JST PH:B12B-PH-K-S
- added C16, C17, C19, C20: 100nF, MyRCL:C-EUC0805
- added D10, D39, D4, D40, D41, D42, D8, D9: BAT54C, diode:BAT54C
- added D13, D14, D15, D16, D18, D19, D20, D21, D31, D32, D33, D34, D35, D36, D37, D38: DDZ9684 (3V3), Diode:ZENER_MMSZ5240BTDO-219-AB(SOD123F)
- added F1, F19, F20, F21, F22, F23, F24: (no value), MyFuse:PTCFUSE-0805
- added IC5: ATAES132A-SHEQ-T, SamacSys_Parts:ATAES132A-SHEQ-T
- added R19, R23, R25, R26: YC164-JR-0733RL, Resistor Array:YC164-JR-0733RL
- added STECKER4: B8B-PH-K-S, con-JST PH:B8B-PH-K-S
- added TVS1, TVS2, TVS4, TVS6, TVS7: USBLC6-4SC6, usblc6:USBLC6-4SC6
- added U1: (no value), microbuilder:EEPROM_I2C_MCP24AA32
- added X5: B10B-PH-KL, con-JST PH:B10B-PH-KL
- F10, F11, F12, F17, F18, F6, F7, F8, F9: value BSMD0805-005-33V -> (none); device rcl:R-EU_R0805 -> MyFuse:PTCFUSE-0805; REICHELT SMD-0805 10,0K -> (none)
- X2: value B7B-PH-K-S -> B10B-PH-KL; device con-JST PH:B7B-PH-K-S -> con-JST PH:B10B-PH-KL
Connections:
- removed net C1_P10: F10.2, STECKER1.10
- removed net C1_P10_F: F10.1, IC2.2, R304.8.1
- removed net C1_P3: F7.2, STECKER1.3
- removed net C1_P3_F: F7.1, IC304.1, R304.3.1
- removed net C1_P4: F8.2, STECKER1.4
- removed net C1_P4_F: F8.1, IC304.2, R304.4.1
- removed net C1_P5: F5.2, STECKER1.5
- removed net C1_P5_F: F5.1, IC303.1, R303.3.1
- removed net C1_P6: F6.2, STECKER1.6
- removed net C1_P6_F: F6.1, IC303.2, R303.4.1
- removed net C1_P7: F4.2, STECKER1.7
- removed net C1_P7_F: F4.1, IC302.1, R302.4.1
- removed net C1_P8: F3.2, STECKER1.8
- removed net C1_P8_F: F3.1, IC302.2, R302.3.1
- removed net C1_P9: F9.2, STECKER1.9
- removed net C1_P9_F: F9.1, IC2.1, R304.7.1
- removed net C2_P10: F18.2, STECKER2.10
- removed net C2_P10_F: F18.1, IC404.1, R404.4.1
- removed net C2_P3: F11.2, STECKER2.3
- removed net C2_P3_F: F12.1, IC401.1, R401.4.1
- removed net C2_P4: F12.2, STECKER2.4
- removed net C2_P4_F: F11.1, IC401.2, R401.3.1
- removed net C2_P5: F14.2, STECKER2.5
- removed net C2_P5_F: F14.1, IC402.1, R402.4.1
- removed net C2_P6: F13.2, STECKER2.6
- removed net C2_P6_F: F13.1, IC402.2, R402.3.1
- removed net C2_P7: F15.2, STECKER2.7
- removed net C2_P7_F: F15.1, IC403.1, R403.3.1
- removed net C2_P8: F16.2, STECKER2.8
- removed net C2_P8_F: F16.1, IC403.2, R403.4.1
- removed net C2_P9: F17.2, STECKER2.9
- removed net C2_P9_F: F17.1, IC404.2, R404.3.1
- removed net EIB_IN: C5.2, IC1.PIO1_8/CT16B1_CAP0, R7.1, T1.E
- removed net IO1: C304.2.2, IC1.PIO2_8/CT32B0_MAT3/TXD, R304.1.2, R304.3.2
- removed net IO10: C401.1.2, IC1.PIO2_2/DCD/MISO1, R401.1.2, R401.3.2
- removed net IO11: C402.1.2, IC1.PIO0_8/MISO0/CT16B0_MAT0, R402.1.2, R402.3.2
- removed net IO12: C402.2.2, IC1.PIO0_9/MOSI0/CT16B0_MAT1, R402.2.2, R402.4.2
- removed net IO13: C403.1.2, IC1.TRST/PIO1_2/AD3/CT32B1_MAT1, R403.1.2, R403.3.2
- removed net IO16: C404.2.2, IC1.TDO/PIO1_1/AD2/CT32B1_MAT0, R404.2.2, R404.4.2
- removed net IO17: IC1.PIO0_4/SCL, R18.1, X2.7
- removed net IO18: IC1.PIO0_5/SDA, R20.1, X2.6
- removed net IO2: C304.1.2, IC1.PIO0_3, R304.2.2, R304.4.2
- removed net IO7: C304.3.2, IC1.PIO2_5/CT32B0_MAT0, R304.5.2, R304.7.2
- removed net IO8: C304.4.2, IC1.PIO3_5/CT16B1_CAP1/TXD, R304.6.2, R304.8.2
- removed net IO9: C401.2.2, IC1.PIO2_10, R401.2.2, R401.4.2
- removed net ISP_EN: IC1.PIO0_1/CLKOUT/CT32B0_MAT2, JP7.7, R15.1
- new net IN1: F9.1, X2.3
- new net IN10: F22.1, X5.4
- new net IN11: F23.1, X5.5
- new net IN12: F24.1, X5.6
- new net IN13: F17.1, X5.7
- new net IN14: F18.1, X5.8
- new net IN15: F19.1, X5.9
- new net IN16: F20.1, X5.10
- new net IN2: F10.1, X2.4
- new net IN3: F11.1, X2.5
- new net IN4: F12.1, X2.6
- new net IN5: F1.1, X2.7
- new net IN6: F6.1, X2.8
- new net IN7: F7.1, X2.9
- new net IN8: F8.1, X2.10
- new net IN9: F21.1, X5.3
- new net IO107: D13.C, D9.A1, IC1.TDI/PIO0_11/AD0/CT32B0_MAT3, R19.8
- new net IO108: D14.C, D9.A2, IC1.TMS/PIO1_0/AD1/CT32B1_CAP0, R19.7
- new net IO109: D10.A1, D15.C, IC1.TDO/PIO1_1/AD2/CT32B1_MAT0, R19.6
- new net IO11/MISO0: IC1.PIO0_8/MISO0/CT16B0_MAT0
- new net IO110: D10.A2, D16.C, IC1.TRST/PIO1_2/AD3/CT32B1_MAT1, R19.5
- new net IO113: C5.2, D35.C, D39.A1, IC1.PIO1_8/CT16B1_CAP0, R26.6, R7.1, T1.E
- new net IO114: D36.C, D39.A2, IC1.PIO0_2/SSEL0/CT16B0_CAP0, R26.5
- new net IO115: D37.C, D40.A1, IC1.PIO2_6/CT32B0_MAT1, R26.8
- new net IO117: D31.C, D41.A1, R25.8
- new net IO118: D32.C, D41.A2, R25.7
- new net IO119: D33.C, D42.A1, R25.6
- new net IO12/MOSI0: IC1.PIO0_9/MOSI0/CT16B0_MAT1
- new net IO120: D34.C, D42.A2, R25.5
- new net IO17/SCL: IC1.PIO0_4/SCL, IC5.SCK, R18.1, STECKER4.3, U1.SCL
- new net IO18/SDA: IC1.PIO0_5/SDA, IC5.SI/SDA, R20.1, STECKER4.4, U1.SDA
- new net ISP_EN/IO116: D38.C, D40.A2, IC1.PIO0_1/CLKOUT/CT32B0_MAT2, JP7.7, R15.1, R26.7
- new net MISO1: IC1.PIO2_2/DCD/MISO1, TVS1.IO3, X3.5
- new net MOSI1: IC1.PIO2_3/RI/MOSI1, TVS1.IO4, X3.6
- new net N$18: F1.2, R19.1, TVS2.IO3
- new net N$19: F6.2, R19.2, TVS2.IO2
- new net N$20: F7.2, R19.3, TVS2.IO1
- new net N$21: F8.2, R19.4, TVS2.IO4
- new net N$22: C16.2, TVS2.VBUS
- new net N$23: F10.2, R23.2, TVS4.IO2
- new net N$24: F12.2, R23.4, TVS4.IO4
- new net N$25: C17.2, TVS4.VBUS
- new net N$26: F11.2, R23.3, TVS4.IO1
- new net N$27: F9.2, R23.1, TVS4.IO3
- new net N$33: F18.2, R25.2, TVS6.IO2
- new net N$34: F20.2, R25.4, TVS6.IO4
- new net N$35: C19.2, TVS6.VBUS
- new net N$36: F19.2, R25.3, TVS6.IO1
- new net N$37: F17.2, R25.1, TVS6.IO3
- new net N$38: F22.2, R26.2, TVS7.IO2
- new net N$39: F24.2, R26.4, TVS7.IO4
- new net N$40: C20.2, TVS7.VBUS
- new net N$42: F23.2, R26.3, TVS7.IO1
- new net N$43: F21.2, R26.1, TVS7.IO3
- new net RXD: IC1.PIO2_7/CT32B0_MAT2/RXD, IC1.PIO3_1/DSR/CT16B0_MAT1/RXD, TVS1.IO1, X3.7
- new net TXD: IC1.PIO2_8/CT32B0_MAT3/TXD, IC1.PIO3_0/DTR/CT16B0_MAT0/TXD, TVS1.IO2, X3.8
- new net XTALOUT: IC1.XTALOUT
- net +3V3: now also D10.CC, D39.CC, D4.CC, D40.CC, D41.CC, D42.CC, D8.CC, D9.CC, IC5.VCC, STECKER4.1, U1.VCC, U1.WP, X2.1, X3.1, X5.1; no longer STECKER1.1, STECKER2.1
- net GND: now also C16.1, C17.1, C19.1, C20.1, D13.A, D14.A, D15.A, D16.A, D18.A, D19.A, D20.A, D21.A, D31.A, D32.A, D33.A, D34.A, D35.A, D36.A, D37.A, D38.A, IC5.VSS, STECKER4.2, TVS1.GND, TVS2.GND, TVS4.GND, TVS6.GND, TVS7.GND, U1.GND, X2.2, X3.2, X5.2; no longer C302.1.1, C302.2.1, C303.1.1, C303.2.1, C304.1.1, C304.2.1, C304.3.1, C304.4.1, C401.1.1, C401.2.1, C402.1.1, C402.2.1, C403.1.1, C403.2.1, C404.1.1, C404.2.1, IC2.3, IC302.3, IC303.3, IC304.3, IC401.3, IC402.3, IC403.3, IC404.3, R302.1.1, R302.2.1, R303.1.1, R303.2.1, R304.1.1, R304.2.1, R304.5.1, R304.6.1, R401.1.1, R401.2.1, R402.1.1, R402.2.1, R403.1.1, R403.2.1, R404.1.1, R404.2.1, STECKER1.2, STECKER2.2
- net IO14: now also IC1.PIO2_1/DSR/SCK1; no longer C403.2.2, IC1.PIO3_0/DTR/CT16B0_MAT0/TXD, R403.2.2, R403.4.2
- net IO15: now also IC1.PIO0_3; no longer C404.1.2, IC1.TMS/PIO1_0/AD1/CT32B1_CAP0, R404.1.2, R404.3.2
- net IO3: now also D20.C, D8.A1, IC1.PIO2_9/CT32B0_CAP0, R23.8; no longer C303.1.2, IC1.PIO0_2/SSEL0/CT16B0_CAP0, R303.1.2, R303.3.2
- net IO4: now also D21.C, D8.A2, IC1.PIO2_10, R23.7; no longer C303.2.2, IC1.PIO2_1/DSR/SCK1, R303.2.2, R303.4.2
- net IO5: now also D18.C, D4.A1, IC1.PIO1_10/AD6/CT16B1_MAT1/MISO1, R23.6; no longer C302.2.2, IC1.PIO2_7/CT32B0_MAT2/RXD, R302.2.2, R302.4.2
- net IO6: now also D19.C, D4.A2, IC1.PIO2_11/SCK0/CT32B0_CAP1, R23.5; no longer C302.1.2, IC1.PIO2_6/CT32B0_MAT1, R302.1.2, R302.3.2
Other:
- moved on the sheet: R18, R20, X3

Commit message: UP Module with fused IOs: alpha version
routing of a version with max. IOs / functions fitting on a single PCB for in-wall installation done. Parts size 0805.
Parts:
- removed IC5: ATAES132A-SHEQ-T, SamacSys_Parts:ATAES132A-SHEQ-T
- removed X3: B8B-PH-K-S, con-JST PH:B8B-PH-K-S
- added C15, C18: 100n, rcl:C-EUC0805
- added CRYPTOIC: ATAES132A-SHER-B, SamacSys_Parts:ATAES132A-SHER-B
- added R17, R24, R27, R28, R29, R30, R40, R41, R42, R43, R44, R45: (no value), rcl:R-EU_R0805
- added R31: 1k, Resistor Array:YC164-JR-0733RL
- added R32, R34: 33R, rcl:R-EU_R0805
- added R33, R35, R36, R37: 100R, rcl:R-EU_R0805
- added R38, R39, R48, R49: 1k, rcl:R-EU_R0805
- added R46, R47: 1K, rcl:R-EU_R0805
- added R50: 100k, rcl:R-EU_R0805
- added R51: 0R0, rcl:R-EU_R0805
- added STECKER3: B8B-PH-K-S, con-JST PH:B8B-PH-K-S
- added TVS3, TVS5, TVS8: USBLC6-4SC6, usblc6:USBLC6-4SC6
- D7: value 3V6 -> DDZ9685 -option; device diode:DIODE-SOD323-R -> microbuilder:DIODESOD-123
- R12: value 91k -> 43k
- R13: value 10k -> 6,2k
- R19, R23, R25, R26: value YC164-JR-0733RL -> (none); device Resistor Array:YC164-JR-0733RL -> rcl:R-EU_R0805
- U1: value (none) -> EEPROM
Connections:
- net N$4 renamed XTALIN
- removed net IO14: IC1.PIO2_1/DSR/SCK1
- removed net IO15: IC1.PIO0_3
- removed net ISP_EN/IO116: D38.C, D40.A2, IC1.PIO0_1/CLKOUT/CT32B0_MAT2, JP7.7, R15.1, R26.7
- removed net RXD: IC1.PIO2_7/CT32B0_MAT2/RXD, IC1.PIO3_1/DSR/CT16B0_MAT1/RXD, TVS1.IO1, X3.7
- removed net TXD: IC1.PIO2_8/CT32B0_MAT3/TXD, IC1.PIO3_0/DTR/CT16B0_MAT0/TXD, TVS1.IO2, X3.8
- new net EIB_IN: C5.2, IC1.PIO0_3, R7.1, T1.E
- new net IN200: R38.2, STECKER3.4
- new net IN201: R39.2, STECKER3.3
- new net IN_MISO1: R35.2, STECKER4.6
- new net IN_MOSI1: R33.2, STECKER4.5
- new net IO116: D38.C, D40.A2, IC1.PIO0_2/SSEL0/CT16B0_CAP0, R43.2
- new net IO19: IC1.PIO3_4/CT16B0_CAP1/RXD, R47.1, TVS8.IO1
- new net IO20: IC1.PIO3_5/CT16B1_CAP1/TXD, R46.1, TVS8.IO2
- new net IO200: IC1.PIO2_3/RI/MOSI1, R39.1, TVS1.IO3
- new net IO201: IC1.PIO1_4/AD5/CT32B1_MAT3/WAKEUP, R38.1, TVS1.IO4
- new net IO21: IC1.PIO0_6/SCK0, R49.1, TVS8.IO4
- new net IO22: IC1.PIO0_7/CTS, R48.1, TVS8.IO3
- new net ISP_EN: IC1.PIO0_1/CLKOUT/CT32B0_MAT2, R15.1, R31.1, TVS3.IO2
- new net N$11: JP7.10, R31.6
- new net N$13: JP7.4, R31.7
- new net N$16: R34.2, STECKER4.4
- new net N$28: Q2.OE, R50.1, R51.2
- new net N$29: R36.2, STECKER3.5
- new net N$30: R37.2, STECKER3.6
- new net N$47: R47.2, STECKER3.8
- new net N$48: R46.2, STECKER3.7
- new net N$49: R49.2, STECKER4.7
- new net N$52: R48.2, STECKER4.8
- new net N$8: JP7.7, R31.5
- new net OLD_REF: D5.C, R3.1, R4.2
- new net RXD2: IC1.PIO3_1/DSR/CT16B0_MAT1/RXD, R36.1, TVS1.IO2
- new net SWD_SWDIO: JP7.2, R31.8
- new net TXD2: IC1.PIO3_0/DTR/CT16B0_MAT0/TXD, R37.1, TVS1.IO1
- new net XTAL_EN: IC1.PIO1_8/CT16B1_CAP0, R51.1
- net +3V3: now also C15.1, C18.1, CRYPTOIC.VCC, R50.2, STECKER3.1, TVS1.VBUS, TVS3.VBUS, TVS5.VBUS, TVS8.VBUS; no longer IC5.VCC, Q2.OE, U1.WP, X3.1
- net EIB_DC: now also D6.C; no longer D5.A
- net EIB_OUT: now also IC1.PIO2_1/DSR/SCK1; no longer IC1.PIO1_9/CT16B1_MAT0/MOSI1
- net GND: now also C15.2, C18.2, CRYPTOIC.CS, CRYPTOIC.VSS, STECKER3.2, TVS3.GND, TVS5.GND, TVS8.GND, U1.WP; no longer IC5.VSS, X3.2
- net IO107: now also R17.2; no longer R19.8
- net IO108: now also R19.2; no longer R19.7
- net IO109: now also R24.2; no longer R19.6
- net IO110: now also R27.2; no longer R19.5
- net IO113: now also IC1.PIO2_7/CT32B0_MAT2/RXD, R44.2; no longer C5.2, IC1.PIO1_8/CT16B1_CAP0, R26.6, R7.1, T1.E
- net IO114: now also IC1.PIO2_8/CT32B0_MAT3/TXD, R45.2; no longer IC1.PIO0_2/SSEL0/CT16B0_CAP0, R26.5
- net IO115: now also R26.2; no longer R26.8
- net IO117: now also R42.2; no longer R25.8
- net IO118: now also R41.2; no longer R25.7
- net IO119: now also R40.2; no longer R25.6
- net IO120: now also R25.2; no longer R25.5
- net IO17/SCL: now also CRYPTOIC.SCK, R34.1, TVS5.IO2; no longer IC5.SCK, STECKER4.3
- net IO18/SDA: now also CRYPTOIC.SI/SDA, R32.1, TVS5.IO1; no longer IC5.SI/SDA, STECKER4.4
- net IO3: now also IC1.PIO2_10, R23.2; no longer IC1.PIO2_9/CT32B0_CAP0, R23.8
- net IO4: now also IC1.PIO2_2/DCD/MISO1, R28.2; no longer IC1.PIO2_10, R23.7
- net IO5: now also R29.2; no longer R23.6
- net IO6: now also R30.2; no longer R23.5
- net MISO1: now also R35.1, TVS5.IO4; no longer IC1.PIO2_2/DCD/MISO1, TVS1.IO3, X3.5
- net MOSI1: now also IC1.PIO1_9/CT16B1_MAT0/MOSI1, R33.1, TVS5.IO3; no longer IC1.PIO2_3/RI/MOSI1, TVS1.IO4, X3.6
- net N$18: now also R17.1; no longer R19.1
- net N$19: now also R19.1; no longer R19.2
- net N$20: now also R24.1; no longer R19.3
- net N$21: now also R27.1; no longer R19.4
- net N$23: now also R28.1; no longer R23.2
- net N$24: now also R30.1; no longer R23.4
- net N$26: now also R29.1; no longer R23.3
- net N$33: now also R41.1; no longer R25.2
- net N$34: now also R25.1; no longer R25.4
- net N$36: now also R40.1; no longer R25.3
- net N$37: now also R42.1; no longer R25.1
- net N$38: now also R43.1; no longer R26.2
- net N$39: now also R45.1; no longer R26.4
- net N$42: now also R44.1; no longer R26.3
- net N$9: now also R32.2, STECKER4.3; no longer D5.C, D6.C
- net REF: now also D5.A; no longer R3.1, R4.2
- net RESET: now also R31.2, TVS3.IO1; no longer JP7.10
- net SWCLK: now also R31.3, TVS3.IO4; no longer JP7.4
- net SWDIO: now also R31.4, TVS3.IO3; no longer JP7.2
Other:
- moved on the sheet: C10, C100, C101, C102, C103, C104, C17, C19, C20, C9, D10, D100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
