File: controller/lpc1115_4te/ARM-LPC1115_V0.08.brd (EAGLE design)
At the start: 66 x 57.9 mm, 53 parts, among them IC1 LPC1115, IC2 MC34063AP, IC3 MCP1702-33, Q1 BC557B, Q3 BC640C, Q4 12MHz, T1 BC547C

Commit message: small changes
Routing:
- net VCC_3V3: track 149.6 -> 143.2 mm
Changed lines of the file:
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@@
 <wire x1="39.4494" y1="52.07" x2="38.3381" y2="52.2288" width="0.254" layer="21"/>
 <wire x1="38.3381" y1="52.2288" x2="40.1638" y2="52.2288" width="0.254" layer="21"/>
-<wire x1="22.5425" y1="30.9563" x2="23.5744" y2="30.9563" width="0.3048" layer="42"/>
 <text x="21.8281" y="2.54" size="1.778" layer="25" rot="R180">LPC1114V0.05</text>
 <text x="43.8944" y="1.8256" size="1.016" layer="27">auf Lötseite:</text>
@@
 <contactref element="IC1" pad="17"/>
 <wire x1="37.2269" y1="36.83" x2="31.75" y2="36.83" width="0.254" layer="16"/>
-<wire x1="31.75" y1="36.83" x2="29.718" y2="34.798" width="0.254" layer="16"/>
-<wire x1="29.718" y1="34.798" x2="29.718" y2="31.75" width="0.254" layer="16"/>
-<wire x1="29.718" y1="31.75" x2="27.813" y2="29.845" width="0.254" layer="16"/>
-<wire x1="27.813" y1="29.845" x2="27.051" y2="29.845" width="0.254" layer="16"/>
-<via x="27.051" y="29.845" extent="1-16" drill="0.6"/>
-<wire x1="26.070625" y1="30.388625" x2="26.070625" y2="31.525625" width="0.254" layer="1"/>
-<wire x1="26.070625" y1="30.388625" x2="26.61425" y2="29.845" width="0.254" layer="1"/>
-<wire x1="26.61425" y1="29.845" x2="27.051" y2="29.845" width="0.254" layer="1"/>
+<wire x1="31.75" y1="36.83" x2="30.988" y2="36.068" width="0.254" layer="16"/>
+<wire x1="26.070625" y1="31.525625" x2="26.070625" y2="30.317375" width="0.254" layer="1"/>
+<wire x1="26.070625" y1="30.317375" x2="26.416" y2="29.972" width="0.254" layer="1"/>
+<wire x1="26.416" y1="29.972" x2="28.067" y2="29.972" width="0.254" layer="1"/>
+<via x="30.988" y="36.068" extent="1-16" drill="0.6"/>
+<wire x1="30.988" y1="36.068" x2="29.337" y2="34.417" width="0.254" layer="1"/>
+<wire x1="29.337" y1="34.417" x2="29.337" y2="32.766" width="0.254" layer="1"/>
+<wire x1="29.337" y1="32.766" x2="28.575" y2="32.004" width="0.254" layer="1"/>
+<wire x1="28.575" y1="32.004" x2="28.575" y2="30.48" width="0.254" layer="1"/>
+<wire x1="28.575" y1="30.48" x2="28.067" y2="29.972" width="0.254" layer="1"/>
 </signal>
 <signal name="EIB+">
@@
 <wire x1="42.6244" y1="46.5931" x2="45.1644" y2="46.5931" width="1.27" layer="1"/>
 <wire x1="42.6244" y1="41.7512" x2="42.6244" y2="46.5931" width="1.27" layer="1"/>
-<polygon width="0.4064" layer="16" isolate="0.254">
+<polygon width="0.4064" layer="16" isolate="25.4">
 <vertex x="-0.1588" y="0"/>
 <vertex x="0" y="59.055"/>
@@
 <vertex x="67.945" y="0"/>
 </polygon>
-<polygon width="0.4064" layer="1" isolate="0.254">
+<polygon width="0.4064" layer="1" isolate="25.4">
 <vertex x="-0.1588" y="59.3725"/>
 <vertex x="-0.1588" y="-0.3175"/>
@@
 <via x="29.21" y="22.098" extent="1-16" drill="0.6"/>
 <wire x1="29.21" y1="22.098" x2="29.21" y2="23.368" width="0.254" layer="1"/>
-<wire x1="29.21" y1="23.368" x2="26.416" y2="26.162" width="0.254" layer="1"/>
-<wire x1="26.416" y1="26.162" x2="22.606" y2="26.162" width="0.254" layer="1"/>
+<wire x1="29.21" y1="23.368" x2="26.924" y2="25.654" width="0.254" layer="1"/>
+<wire x1="26.924" y1="25.654" x2="23.114" y2="25.654" width="0.254" layer="1"/>
 <wire x1="22.062375" y1="27.975625" x2="21.020625" y2="27.975625" width="0.254" layer="1"/>
 <wire x1="22.062375" y1="27.975625" x2="22.352" y2="27.686" width="0.254" layer="1"/>
 <wire x1="22.352" y1="27.686" x2="22.352" y2="26.416" width="0.254" layer="1"/>
-<wire x1="22.352" y1="26.416" x2="22.606" y2="26.162" width="0.254" layer="1"/>
+<wire x1="22.352" y1="26.416" x2="23.114" y2="25.654" width="0.254" layer="1"/>
 </signal>
 <signal name="IO3">
@@
 <contactref element="IC1" pad="13"/>
 <contactref element="SV1" pad="1"/>
-<wire x1="28.070625" y1="31.525625" x2="28.070625" y2="31.880625" width="0.254" layer="1"/>
+<wire x1="28.070625" y1="31.525625" x2="28.070625" y2="32.261625" width="0.254" layer="1"/>
 <via x="29.337" y="36.83" extent="1-16" drill="0.6"/>
 <wire x1="29.337" y1="36.83" x2="22.86" y2="36.83" width="0.254" layer="16"/>
 <wire x1="22.86" y1="36.83" x2="20.066" y2="34.036" width="0.254" layer="16"/>
 <wire x1="20.066" y1="34.036" x2="18.034" y2="34.036" width="0.254" layer="16"/>
-<wire x1="28.070625" y1="31.880625" x2="29.337" y2="33.147" width="0.254" layer="1"/>
-<wire x1="29.337" y1="33.147" x2="29.337" y2="36.83" width="0.254" layer="1"/>
 <wire x1="18.034" y1="34.036" x2="13.890625" y2="38.179375" width="0.254" layer="16"/>
 <wire x1="13.890625" y1="38.179375" x2="13.509625" y2="38.179375" width="0.254" layer="16"/>
+<wire x1="28.070625" y1="32.261625" x2="28.829" y2="33.02" width="0.254" layer="1"/>
+<wire x1="28.829" y1="33.02" x2="28.829" y2="35.179" width="0.254" layer="1"/>
+<wire x1="28.829" y1="35.179" x2="29.337" y2="35.687" width="0.254" layer="1"/>
+<wire x1="29.337" y1="35.687" x2="29.337" y2="36.83" width="0.254" layer="1"/>
 </signal>
 <signal name="LT2">
@@
 <wire x1="18.478625" y1="42.608625" x2="18.259525" y2="42.608625" width="1.016" layer="16"/>
 <wire x1="38.1476" y1="31.2419" x2="38.1476" y2="31.1944" width="1.016" layer="16"/>
-<wire x1="38.1476" y1="31.1944" x2="41.402" y2="27.94" width="1.016" layer="16"/>
-<wire x1="41.402" y1="27.94" x2="41.402" y2="24.892" width="1.016" layer="16"/>
-<wire x1="41.402" y1="24.892" x2="38.862" y2="22.352" width="1.016" layer="16"/>
-<wire x1="38.862" y1="22.352" x2="35.56" y2="22.352" width="1.016" layer="16"/>
-<wire x1="35.56" y1="22.352" x2="34.798" y2="21.59" width="1.016" layer="16"/>
-<wire x1="34.798" y1="21.59" x2="34.798" y2="16.51" width="1.016" layer="16"/>
-<wire x1="34.798" y1="16.51" x2="35.90925" y2="15.65275" width="1.016" layer="16"/>
-<wire x1="35.90925" y1="15.65275" x2="39.08475" y2="15.66875" width="1.016" layer="16"/>
+<wire x1="38.1476" y1="31.1944" x2="40.132" y2="28.956" width="1.016" layer="16"/>
+<wire x1="40.132" y1="28.956" x2="40.132" y2="23.622" width="1.016" layer="16"/>
+<wire x1="40.132" y1="23.622" x2="37.084" y2="20.574" width="1.016" layer="16"/>
 <wire x1="39.08475" y1="15.66875" x2="38.1" y2="15.5575" width="1.016" layer="16"/>
 <wire x1="38.1" y1="15.5575" x2="38.1" y2="14.986" width="1.016" layer="16"/>
@@
 <wire x1="32.004" y1="16.256" x2="38.4975" y2="16.256" width="1.016" layer="1"/>
 <wire x1="38.4975" y1="16.256" x2="39.08475" y2="15.66875" width="1.016" layer="1"/>
+<wire x1="37.084" y1="20.574" x2="37.084" y2="16.764" width="1.016" layer="16"/>
+<wire x1="37.084" y1="16.764" x2="38.17925" y2="15.66875" width="1.016" layer="16"/>
+<wire x1="38.17925" y1="15.66875" x2="39.08475" y2="15.66875" width="1.016" layer="16"/>
 </signal>
 <signal name="VCC_A">
