File: controller/lpc1115_2te/LPC1115_2TE_V1.02.brd (EAGLE design)
At the start: 30.5 x 58.1 mm, 57 parts, among them IC1 LPC1115, IC2 BD9G101, Q1 BC856, Q2 BC847C, Q3 BCP52, Q4 ASFL

Commit message: GND Plane optimiert
Routing:
- net SWCLK: track 18.2 -> 19.6 mm
- net GND: vias 29 -> 30
Other:
- board text added: "Ref"
