File: applications/out6_cs/ou6_cs-ctrl V1.0.brd (EAGLE design)
At the start: 100 x 58 mm, 82 parts, among them P3 SE1.5, P4 SE1.5, P5 SE1.5, Q1 BCP52, T1 AX1500, T2 AX1500, T3 AX1500, T4 AX1500, T5 AX1500, T6 AX1500, U1 74LV4051D, U2 OPA365AIDBV, U3 OPA365AIDBV, U4 OPA340NA

Commit message: Update App out6_cs, update Controller lpc1115_4te_top
Parts:
- U4: value OPA340NA -> OPA365AIDBV
Changed lines of the file:
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@@
 <attribute name="VALUE" x="49.8758" y="21.9544" size="1.27" layer="27" ratio="6" rot="R270"/>
 </element>
-<element name="U4" library="eigene" package="SOT23-5" value="OPA340NA" x="35" y="29.5" smashed="yes">
+<element name="U4" library="eigene" package="SOT23-5" value="OPA365AIDBV" x="35" y="29.5" smashed="yes">
 <attribute name="NAME" x="31.394" y="29.995" size="1.27" layer="25" ratio="12" rot="R180"/>
 <attribute name="VALUE" x="31.5456" y="26.3758" size="1.27" layer="27" ratio="6"/>
