File: applications/out6_cs/ou6_cs-ctrl V1.1.brd (EAGLE design)
At the start: 100 x 57 mm, 83 parts, among them P3 SE1.5, P4 SE1.5, P5 SE1.5, Q1 BCP52, T1 AX1500, T2 AX1500, T3 AX1500, T4 AX1500, T5 AX1500, T6 AX1500, U1 74LV4051D, U2 OPA365AIDBV, U3 OPA365AIDBV, U4 OPA365AIDBV

Commit message: R29 auf out6_cs-ctrl V1.1 auf unbestückt geändert
Parts:
- R29: value 100k -> -
Changed lines of the file:
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@@
 <attribute name="VALUE" x="79.135" y="14.04" size="1.27" layer="27" rot="R180"/>
 </element>
-<element name="R29" library="rcl" package="R0805M" value="100k" x="42" y="19.5"/>
+<element name="R29" library="rcl" package="R0805M" value="-" x="42" y="19.5"/>
 </elements>
 <signals>
