File: applications/2out_16A_bi_TS/2out_16A_bi_TS-ARM_V1.0.brd (EAGLE design)
At the start: 42.3 x 27.4 mm, 31 parts, among them K1 HFE20-1/024-1HD-L2, K2 HFE20-1/024-1HD-L2, T1 BC847, T2 BC847, T3 BC847, T4 BC847

Commit message: Spannungsteiler auf 91k/10k geändert
Parts:
- R6: value 36K 1% -> 91K 1%
- R7: value 3K 1% -> 10K 1%
Changed lines of the file:
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@@
 <attribute name="VALUE" x="5.23215625" y="20.85779375" size="1.27" layer="27" rot="R180"/>
 </element>
-<element name="R6" library="rcl" package="M1206" value="36K 1%" x="5.715" y="17.4625" smashed="yes">
+<element name="R6" library="rcl" package="M1206" value="91K 1%" x="5.715" y="17.4625" smashed="yes">
 <attribute name="NAME" x="8.5725" y="17.78" size="0.8128" layer="25"/>
 <attribute name="VALUE" x="10.4775" y="17.78" size="0.8128" layer="27"/>
 </element>
-<element name="R7" library="rcl" package="M1206" value="3K 1%" x="4.28625" y="22.38375" smashed="yes" rot="MR90">
+<element name="R7" library="rcl" package="M1206" value="10K 1%" x="4.28625" y="22.38375" smashed="yes" rot="MR90">
 <attribute name="NAME" x="2.2225" y="22.225" size="0.8128" layer="26" rot="MR90"/>
 <attribute name="VALUE" x="1.27" y="21.59" size="0.8128" layer="28" rot="MR90"/>
